Commit message: add ee_link

File: ur_description/urdf/ur_macro.xacro (robot description, xacro)
@@ -308,10 +308,16 @@
       <origin xyz="0 0 0" rpy="0 ${-pi/2.0} ${-pi/2.0}" />
     </joint>
+    <link name="${prefix}ee_link" />
+    <joint name="${prefix}frange-ee_link" type="fixed">
+      <parent link="${prefix}flange" />
+      <child link="${prefix}ee_link" />
+      <origin xyz="0 0 0" rpy="${pi} 0 0" />
+    </joint>
     <!-- ROS-Industrial 'tool0' frame: all-zeros tool frame -->
     <link name="${prefix}tool0"/>
-    <joint name="${prefix}flange-tool0" type="fixed">
+    <joint name="${prefix}ee_link-tool0" type="fixed">
       <!-- default toolframe: X+ left, Y+ up, Z+ front -->
-      <origin xyz="0 0 0" rpy="${pi/2.0} 0 ${pi/2.0}"/>
-      <parent link="${prefix}flange"/>
+      <origin xyz="0 0 0" rpy="${-pi/2.0} 0 ${-pi/2.0}"/>
+      <parent link="${prefix}ee_link"/>
       <child link="${prefix}tool0"/>
     </joint>
